Commit message: Update turtlebot3_burger_cam model: Adjust camera pose and horizontal field of view for improved accuracy

File: src/turtlebot3_simulations/turtlebot3_gazebo/urdf/turtlebot3_burger_cam.urdf (robot description, URDF)
Before this commit: robot turtlebot3_burger_cam, 10 links, 9 joints
Joints:
- joint camera_joint: origin xyz=0.040 -0.000 0.110 rpy=0 0 0 -> xyz=0.040 -0.000 0.128 rpy=0 0.524 0
